File: design/buttons.kicad_sch (KiCad schematic)
At the start: 32 parts, among them SW201 SW_Push, SW202 SW_Push, SW203 SW_Push, SW204 SW_Push, SW205 SW_Push, SW206 SW_Push, SW207 SW_Push, SW208 SW_Push, SW209 SW_Push, SW210 SW_Push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

Commit message: start layout
Parts:
- removed D201, D202, D203, D204, D205, D206, D207, D208, D209, D210, D211, D212, D213, D214, D215, D216: D, symbol Device:D
- added D201, D202, D203, D204, D205, D206, D207, D208, D209, D210, D211, D212, D213, D214, D215, D216: 1N5819W, Diode_SMD:D_SOD-123F, symbol Device:D_Schottky
Connections:
- net COL0: now also D201.1 (K), D205.1 (K), D209.1 (K), D213.1 (K)
- net COL1: now also D202.1 (K), D206.1 (K), D210.1 (K), D214.1 (K)
- net COL2: now also D203.1 (K), D207.1 (K), D211.1 (K), D215.1 (K)
- net COL3: now also D204.1 (K), D208.1 (K), D212.1 (K), D216.1 (K)
- net at SW207.1: now also D207.2 (A)
- net at SW212.1: now also D212.2 (A)
- net at SW211.1: now also D211.2 (A)
- net at SW210.1: now also D210.2 (A)
- net at SW216.1: now also D216.2 (A)
- net at SW209.1: now also D209.2 (A)
- net at SW206.1: now also D206.2 (A)
- net at SW205.1: now also D205.2 (A)
- net at SW208.1: now also D208.2 (A)
- net at SW214.1: now also D214.2 (A)
- net at SW204.1: now also D204.2 (A)
- net at SW201.1: now also D201.2 (A)
- net at SW203.1: now also D203.2 (A)
- net at SW215.1: now also D215.2 (A)
- net at SW213.1: now also D213.2 (A)
- net at SW202.1: now also D202.2 (A)
