File: design/controller.kicad_pcb (KiCad board)
At the start: 2 copper layers, 104 x 241 mm, 68 parts, among them J101 2.1x5.5mm, J102 Screw_Terminal_01x05, J103 Screw_Terminal_01x05, J104 Screw_Terminal_01x05, J105 MIKROBUS_MODULE, J106 XLR5_Ground, J107 Conn_01x02, J108 Conn_01x02, SW201 SW_Push, SW202 SW_Push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

Commit message: routing
Parts:
- C101, C102, C103, C104, C105, C106, C107, C108, C109, D101, D102, FB101, FB102, J102, J103, J104, JP101, JP102, R101, U102, U103, U104, U106: moved to B.Cu
- moved D101 160.2 mm to (57.8, -19.7), turned to 180 degrees
- moved JP102 146.3 mm to (53.3, -5.34), turned to 180 degrees
- moved JP101 146.3 mm to (53.3, -8.89), turned to 180 degrees
- moved C104 142.9 mm to (78.7, 170.8)
- moved D102 142.5 mm to (14.0, -15.9), turned to 180 degrees
- moved C103 140.3 mm to (71.8, 170.8)
- moved C102 138.1 mm to (64.8, 170.8)
- moved C109 126.5 mm to (78.7, 161.3), turned to 180 degrees
- moved C108 123.4 mm to (71.8, 161.9), turned to 180 degrees
- moved C107 120.3 mm to (64.8, 161.9), turned to 180 degrees
- moved FB102 117.4 mm to (-3.81, -22.2), turned to 180 degrees
- moved R101 117.0 mm to (26.0, -9.53), turned to 180 degrees
- moved FB101 115.9 mm to (3.17, -22.2), turned to 180 degrees
- moved C101 107.2 mm to (17.1, -40.0)
- moved C105 105.2 mm to (16.5, -26.0)
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Routing:
- net /BUTTONS_COL2: track 0.00 -> 173.1 mm
- net /BUTTONS_COL1: track 0.00 -> 173.0 mm
- net /BUTTONS_COL0: track 0.00 -> 173.0 mm
- net /BUTTONS_COL3: track 0.00 -> 60.0 mm
- net /BUTTONS_ROW3: track 0.00 -> 40.0 mm
- net /BUTTONS_ROW2: track 0.00 -> 40.0 mm
- net /BUTTONS_ROW1: track 0.00 -> 40.0 mm
- net /BUTTONS_ROW0: track 0.00 -> 40.0 mm
- net Net-(D214-A): track 0.00 -> 4.48 mm
- net Net-(D210-A): track 0.00 -> 4.48 mm
- net Net-(D213-A): track 0.00 -> 4.48 mm
- net Net-(D209-A): track 0.00 -> 4.48 mm
- net Net-(D215-A): track 0.00 -> 4.48 mm
- net Net-(D211-A): track 0.00 -> 4.48 mm
- net Net-(D205-A): track 0.00 -> 4.48 mm
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- added copper zone on F.Cu, net +5V
- added copper zone on B.Cu, net GND

Commit message: final design
Parts:
- added G***: LOGO, LOGO, F.Cu at (39.5, 35.3)
- added G***: LOGO, LOGO, F.Cu at (21.8, 109.0)
- added G***: LOGO, LOGO, F.Cu at (2.51, 0.03)
- added G***: LOGO, LOGO, F.Cu at (49.2, 82.2)
- added G***: LOGO, LOGO, F.Cu at (35.3, 144.3)
- added G***: LOGO, LOGO, F.Cu at (20.0, -23.0)
- added REF**: MountingHole_2.2mm_M2, MountingHole:MountingHole_2.2mm_M2, F.Cu at (-7.00, -38.5)
- added REF**: MountingHole_2.2mm_M2, MountingHole:MountingHole_2.2mm_M2, F.Cu at (91.0, -38.5)
- added REF**: MountingHole_2.2mm_M2, MountingHole:MountingHole_2.2mm_M2, F.Cu at (91.0, 196.5)
- added REF**: MountingHole_2.2mm_M2, MountingHole:MountingHole_2.2mm_M2, F.Cu at (-7.00, 196.5)
- moved D102 183.9 mm to (75.2, 157.5), turned to 0 degrees
- moved J105 178.6 mm to (66.8, 172.9), turned to 0 degrees
- moved JP101 177.8 mm to (73.3, 167.8), turned to 0 degrees
- moved JP102 171.8 mm to (73.3, 165.2), turned to 0 degrees
- moved C102 147.1 mm to (71.0, 23.9)
- moved U102 139.9 mm to (73.0, 26.1)
- moved C107 138.4 mm to (75.0, 23.9)
- moved C103 133.0 mm to (71.0, 37.8)
- moved J102 131.1 mm to (79.0, 17.3)
- moved U103 125.7 mm to (73.0, 40.1)
- moved C108 124.1 mm to (75.0, 37.8)
- moved C104 119.4 mm to (71.0, 51.6)
- moved J103 116.9 mm to (79.0, 31.3)
- moved U104 111.8 mm to (73.0, 54.0)
- moved C109 109.7 mm to (75.0, 51.6)
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Connections:
- U101 pad 12: /BUTTONS_COL0 -> unconnected-(U101-GPIO9-Pad12)
- U101 pad 15: /BUTTONS_COL1 -> unconnected-(U101-GPIO11-Pad15)
- U101 pad 19: /BUTTONS_COL2 -> unconnected-(U101-GPIO14-Pad19)
- U101 pad 24: unconnected-(U101-GPIO18-Pad24) -> /BUTTONS_COL2
- U101 pad 25: unconnected-(U101-GPIO19-Pad25) -> /BUTTONS_COL1
- U101 pad 29: unconnected-(U101-GPIO22-Pad29) -> /BUTTONS_COL0
Routing:
- net /BUTTONS_ROW2: track 40.0 -> 260.5 mm
- net +10V: track 0.00 -> 211.7 mm, vias 0 -> 10
- net /BUTTONS_ROW3: track 40.0 -> 232.1 mm
- net /UART0_RX: track 0.00 -> 177.9 mm
- net /UART0_TX: track 0.00 -> 177.8 mm
- net /BUTTONS_ROW0: track 40.0 -> 188.5 mm, vias 0 -> 2
- net /BUTTONS_ROW1: track 40.0 -> 181.9 mm, vias 0 -> 1
- net +3.3V: track 0.00 -> 102.1 mm, vias 0 -> 1
- net GND: track 0.00 -> 91.0 mm, vias 0 -> 17
- net /FADER2_LEVEL: track 0.00 -> 82.1 mm
- net /FADER2_PWM0: track 0.00 -> 81.4 mm
- net /FADER1_PWM0: track 0.00 -> 79.3 mm
- net /WS2811_1: track 0.00 -> 77.8 mm
- net /FADER0_PWM1: track 0.00 -> 77.3 mm
- net /BUTTONS_COL3: track 60.0 -> 135.1 mm, vias 0 -> 1
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- added copper zone on F.Cu, net +3.3V
- added copper zone on B.Cu, net +5V
- added copper zone on B.Cu, net Net-(FB101-Pad2)
- added copper zone on B.Cu, net Net-(FB102-Pad1)
Other:
- outline, holes or cut-outs redrawn
- board text added: "Hinkle Inc."
