File: design/controller.kicad_sch (KiCad schematic)
At the start: 30 parts, among them J101 Barrel_Jack, J102 Screw_Terminal_01x05, J103 Screw_Terminal_01x05, J104 Screw_Terminal_01x05, J105 MIKROBUS_MODULE, J106 XLR5_Ground, J107 Conn_01x02, J108 Conn_01x02, U101 Pico, U102 DRV8837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

Commit message: start layout
Parts:
- added H101, H102, H103, H104, H105, H106: M3x0.5, MountingHole:MountingHole_3.2mm_M3_DIN965_Pad_TopBottom, symbol Mechanical:MountingHole
- D101, D102: value D_Schottky -> 1N5819W; footprint (none) -> Diode_SMD:D_SOD-123F
- FB101, FB102: footprint (none) -> Resistor_SMD:R_0805_2012Metric_Pad1.20x1.40mm_HandSolder
- J101: value Barrel_Jack -> 2.1x5.5mm; footprint (none) -> Connector_BarrelJack:BarrelJack_CUI_PJ-063AH_Horizontal
- J102, J103, J104: footprint (none) -> Connector_PinHeader_2.54mm:PinHeader_1x05_P2.54mm_Vertical
- U105: footprint (none) -> Package_TO_SOT_SMD:TO-263-2
Connections:
- net UART1_RX: no longer U106.4 (DI)
- net UART1_TX: now also U106.4 (DI)

Commit message: final design
Connections:
- net BUTTONS_COL0: now also U101.29 (GPIO22); no longer U101.12 (GPIO9)
- net BUTTONS_COL1: now also U101.25 (GPIO19); no longer U101.15 (GPIO11)
- net BUTTONS_COL2: now also U101.24 (GPIO18); no longer U101.19 (GPIO14)
Changed lines of the file:
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@@
 	(wire
 		(pts
-			(xy 80.01 111.76) (xy 99.06 111.76)
+			(xy 153.67 106.68) (xy 134.62 106.68)
 		)
 		(stroke
@@
 	(wire
 		(pts
-			(xy 80.01 101.6) (xy 99.06 101.6)
+			(xy 153.67 104.14) (xy 134.62 104.14)
 		)
 		(stroke
@@
 	(wire
 		(pts
-			(xy 80.01 93.98) (xy 99.06 93.98)
+			(xy 153.67 93.98) (xy 134.62 93.98)
 		)
 		(stroke
@@
 	)
 	(label "BUTTONS_COL0"
-		(at 80.01 93.98 0)
-		(fields_autoplaced yes)
-		(effects
-			(font
-				(size 1.27 1.27)
-			)
-			(justify left bottom)
+		(at 153.67 93.98 180)
+		(fields_autoplaced yes)
+		(effects
+			(font
+				(size 1.27 1.27)
+			)
+			(justify right bottom)
 		)
 	)
@@
 	)
 	(label "BUTTONS_COL2"
-		(at 80.01 111.76 0)
-		(fields_autoplaced yes)
-		(effects
-			(font
-				(size 1.27 1.27)
-			)
-			(justify left bottom)
+		(at 153.67 106.68 180)
+		(fields_autoplaced yes)
+		(effects
+			(font
+				(size 1.27 1.27)
+			)
+			(justify right bottom)
 		)
 	)
@@
 	)
 	(label "BUTTONS_COL1"
-		(at 80.01 101.6 0)
-		(fields_autoplaced yes)
-		(effects
-			(font
-				(size 1.27 1.27)
-			)
-			(justify left bottom)
-		)
-	)
+		(at 153.67 104.14 180)
+		(fields_autoplaced yes)
+		(effects
+			(font
+				(size 1.27 1.27)
+			)
+			(justify right bottom)
+		)
+	)
